Commit message: added stock joint limits from universal robots package

File: ur5e_with_robotiq/ur5e_with_robotiq/urdf/ur5e_with_robotiq.urdf (robot description, URDF)
Before this commit: robot ur5e_with_soft_hand, 13 links, 12 joints
Joints:
- joint world_joint: origin xyz=0.0 0.0 0.0 rpy=0.0 0.0 0.0 -> xyz=0.0 0.0 0.0 rpy=0.0 0.0 0.0349066

File: ur5e_with_robotiq/ur5e_with_robotiq/urdf/ur5e_with_robotiq.xacro (robot description, xacro)
@@ -17,5 +17,5 @@
     <parent link="world" />
     <child link="base_link" /> <!-- TODO: check base_link name of robot -->
-    <origin xyz="0.0 0.0 0.0" rpy="0.0 0.0 0.0" />
+    <origin xyz="0.0 0.0 0.0" rpy="0.0 0.0 0.0349066" />
   </joint>
 </robot>

File: ur5e_with_soft_hand/ur5e_with_soft_hand/urdf/ur5e_with_soft_hand.urdf (robot description, URDF)
Before this commit: robot ur5e_with_soft_hand, 13 links, 12 joints
Joints:
- joint world_joint: origin xyz=0.0 0.0 0.0 rpy=0.0 0.0 0.0 -> xyz=0.0 0.0 0.0 rpy=0.0 0.0 0.0349066
